File: hardware/tht/ttl2dvi_tht.kicad_pcb (KiCad board)
At the start: 2 copper layers, 88 x 88 mm, 40 parts, among them J1 RP2350-PiZero, J2 DE9 male (video in), J3 IDC10 (alt video in), J4 Logic analyser, J5 Console, J6 5V IN, SW1 PREV, SW2 NEXT, SW3 ENTER, U1 74LVC245A / 74HCT541, U2 74LVC14A / 74HCT14, U3 VS1838B

Commit message: update tht design - move console pins
Parts:
- removed TP1: 3V3, TestPoint:TestPoint_THTPad_D2.0mm_Drill1.0mm
- removed TP2: GND, TestPoint:TestPoint_THTPad_D2.0mm_Drill1.0mm
- removed TP4: 5V, TestPoint:TestPoint_THTPad_D2.0mm_Drill1.0mm
- moved J5 76.5 mm to (179.9, 53.8)
- moved R11 35.8 mm to (177.3, 71.2), turned to 90 degrees
- moved R12 35.8 mm to (173.0, 71.2), turned to 90 degrees
Routing:
- net /TX: track 43.1 -> 12.5 mm, vias 1 -> 0
- net +5V: track 68.7 -> 43.3 mm
- net /RX: track 42.5 -> 21.5 mm
- net +3V3: track 89.2 -> 78.4 mm
- net Net-(J5-Pin_2): track 16.5 -> 9.82 mm
- net Net-(J5-Pin_3): track 16.2 -> 10.5 mm
- net /GP23: track 41.5 -> 44.9 mm, vias 2 -> 4
- net /GP24: track 42.0 -> 43.2 mm, vias 2 -> 3
- net /GP25: track 38.2 -> 39.1 mm, vias 2 -> 3
- net /GP22: vias 4 -> 3
Other:
- board text added: "pico-ttl2dvi THT rev A"
- board text removed: "3.3V"
- board text removed: "TP1"
- board text removed: "TP4"
- board text removed: "pico-ttl2dvi THT rev X1"
