File: hardware/tht/ttl2dvi_tht.kicad_sch (KiCad schematic)
At the start: 40 parts, among them J1 RP2350-PiZero, J2 DE9 male (video in), J3 IDC10 (alt video in), J4 Logic analyser, J5 Console, J6 5V IN, SW1 PREV, SW2 NEXT, SW3 ENTER, U1 74LVC245A / 74HCT541, U2 74LVC14A / 74HCT14, U3 VS1838B

Commit message: update tht design - move console pins
Parts:
- removed TP1: 3V3, TestPoint:TestPoint_THTPad_D2.0mm_Drill1.0mm, symbol Connector:TestPoint
- removed TP2: GND, TestPoint:TestPoint_THTPad_D2.0mm_Drill1.0mm, symbol Connector:TestPoint
- removed TP4: 5V, TestPoint:TestPoint_THTPad_D2.0mm_Drill1.0mm, symbol Connector:TestPoint
