File: hardware/tht/revA/ttl2dvi_tht.kicad_sch (KiCad schematic)
At the start: 37 parts, among them J1 RP2350-PiZero, J2 DE9 male (video in), J3 IDC10 (alt video in), J4 Logic analyser, J5 Console, J6 5V IN, SW1 PREV, SW2 NEXT, SW3 ENTER, U1 74LVC245A / 74HCT541, U2 74LVC14A / 74HCT14, U3 VS1838B

Commit message: update tht reva hardware design
Parts:
- H1, H2, H3, H4: footprint MountingHole:MountingHole_3.2mm_M3_Pad -> MountingHole:MountingHole_3.2mm_M3_Pad_Via
Changed lines of the file:
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@@
 	(title_block
 		(title "ttl2dvi throughole baseboard")
-		(rev "THT X1")
+		(rev "THT A")
 	)
 	(text_box "WAVESHARE BOARD"
@@
 			)
 		)
-		(property "Footprint" "MountingHole:MountingHole_3.2mm_M3_Pad"
+		(property "Footprint" "MountingHole:MountingHole_3.2mm_M3_Pad_Via"
 			(at 173.99 247.65 0)
 			(hide yes)
@@
 			)
 		)
-		(property "Footprint" "MountingHole:MountingHole_3.2mm_M3_Pad"
+		(property "Footprint" "MountingHole:MountingHole_3.2mm_M3_Pad_Via"
 			(at 173.99 261.62 0)
 			(hide yes)
@@
 			)
 		)
-		(property "Footprint" "MountingHole:MountingHole_3.2mm_M3_Pad"
+		(property "Footprint" "MountingHole:MountingHole_3.2mm_M3_Pad_Via"
 			(at 161.29 247.65 0)
 			(hide yes)
@@
 			)
 		)
-		(property "Footprint" "MountingHole:MountingHole_3.2mm_M3_Pad"
+		(property "Footprint" "MountingHole:MountingHole_3.2mm_M3_Pad_Via"
 			(at 161.29 261.62 0)
 			(hide yes)
